File: electrical/BMS/BMS_vtest/BMS_vtest.kicad_sch (KiCad schematic)
At the start: 77 parts, among them Q1 NMOS, Q2 NPN, U1 STM32F103C4Tx, U2 BQ79612PAPRQ1

Commit message: more components yay!
Parts:
- removed U1: STM32F103C4Tx, Package_QFP:LQFP-48_7x7mm_P0.5mm, symbol MCU_ST_STM32F1:STM32F103C4Tx
- added R37: 10k, symbol Device:R
- added TH3: Thermistor_NTC, symbol Device:Thermistor_NTC
- added U3: CD74HC4067M, Package_SO:SOIC-24W_7.5x15.4mm_P1.27mm, symbol 74xx:CD74HC4067M
- added U4: STM32F103C6Tx, Package_QFP:LQFP-48_7x7mm_P0.5mm, symbol MCU_ST_STM32F1:STM32F103C6Tx
Connections:
- net TSREF is gone; now on net GPIO2: C35.1, R34.1, R35.1, U2.51
- net AFE_RX: now also U4.30 (PA9)
- net AFE_TX: now also U4.31 (PA10)
- net AVDD: now also U3.24 (VCC)
- net GND: now also TH3.2
- net GPIO2: now also U2.60, R37.1
- net GPIO3: now also U2.59, R37.2, TH3.1; no longer R35.2, R36.1, TH2.1
- net VDD1: now also U4.24 (VDD)
- net GPIO4: now reaches U2.58
- net GPIO4: now also R35.2, R36.1, TH2.1
- new net: U4.23 (VSS), U4.35 (VSS), U4.47 (VSS)
Other:
- note added: "MOSFET (2) Ambient Temperature (3) PCB Cell Balancing (4)"
- note removed: "MOSFET (2) and PCB Cell Balancing (3)"
- moved on the sheet: C35, R34, TH1
